File: 04_test_and_results/first_motor_control/Electronics/motor_control/motor_control.kicad_sch (KiCad schematic)
At the start: 11 parts, among them J2 Conn_01x03_Pin, Q1 BD909, Q2 BD909, Q3 BD909, Q4 BD909, Q5 BD909, Q6 BD909, U1 STM32F103C6T6

Commit message: update
Parts:
- removed D1: LED, symbol Device:LED
- added D2, D3, D4, D5, D6, D7: D, symbol Device:D
Connections:
- net GNDP: now also D4.2 (A), D5.2 (A), D6.2 (A)
- net VCCP: now also D2.1 (K), D3.1 (K), D7.1 (K)
- net at J2.2 (Pin_2), Q3.3 (E), Q4.2 (C): now also D2.2 (A), D5.1 (K)
- net at J2.3 (Pin_3), Q5.3 (E), Q6.2 (C): now also D3.2 (A), D4.1 (K)
- net at J2.1 (Pin_1), Q1.3 (E), Q2.2 (C): now also D6.1 (K), D7.2 (A)
Other:
- moved on the sheet: J2, Q1, Q2, Q5, Q6
